Commit message: Change rocker joints to revolute

File: description/rover.urdf (robot description, URDF)
Before this commit: robot rover, 11 links, 10 joints
Joints:
- joint left_rocker_joint: limit (none) -> lower=-0.548 upper=0.548 effort=1000.0 velocity=0.5; type continuous -> revolute
- joint right_rocker_joint: limit (none) -> lower=-0.548 upper=0.548 effort=1000.0 velocity=0.5; type continuous -> revolute

Commit message: Added lidar to simulation

File: description/rover.urdf (robot description, URDF)
Before this commit: robot rover, 11 links, 10 joints
Links:
- added link laser_frame, mass 0.1; collision cylinder length=0.04 radius=0.05; visual cylinder length=0.04 radius=0.05
Joints:
- added joint laser_joint: type fixed, parent frame, child laser_frame, origin xyz=0 -0.4 .37 rpy=0 0 0

Commit message: Removed extra rover urdf file and added two cameras: normal and depth

File: description/rover.urdf (robot description, URDF)
Before this commit: robot rover, 12 links, 11 joints
Links:
- added link camera_link; visual box size=0.010 0.03 0.03
- added link camera_link_optical
Joints:
- added joint camera_joint: type fixed, parent frame, child camera_link, origin xyz=0 .5 .37 rpy=0 0 1.57
- added joint camera_optical_joint: type fixed, parent camera_link, child camera_link_optical, origin xyz=0 0 0 rpy=${-pi/2} 0 ${-pi/2}
